Commit message: [chore] update new description

File: navexbot_description/navexbot_description/urdf/materials.xacro (robot description, xacro)
@@ -1,4 +1,4 @@
 <?xml version="1.0" ?>
-<robot name="Elegoo_to_urdf" xmlns:xacro="http://www.ros.org/wiki/xacro" >
+<robot name="navexbot" xmlns:xacro="http://www.ros.org/wiki/xacro" >
 <material name="silver">
   <color rgba="0.700 0.700 0.700 1.000"/>

File: navexbot_description/navexbot_description/urdf/navexbot.xacro (robot description, xacro)
@@ -1,17 +1,17 @@
 <?xml version="1.0" ?>
-<robot name="Elegoo_to_urdf" xmlns:xacro="http://www.ros.org/wiki/xacro">
-<xacro:include filename="$(find Elegoo_to_urdf_description)/urdf/materials.xacro" />
-<xacro:include filename="$(find Elegoo_to_urdf_description)/urdf/Elegoo_to_urdf.trans" />
-<xacro:include filename="$(find Elegoo_to_urdf_description)/urdf/Elegoo_to_urdf.gazebo" />
+<robot name="navexbot" xmlns:xacro="http://www.ros.org/wiki/xacro">
+<xacro:include filename="$(find navexbot_description)/urdf/materials.xacro" />
+<xacro:include filename="$(find navexbot_description)/urdf/navexbot.trans" />
+<xacro:include filename="$(find navexbot_description)/urdf/navexbot.gazebo" />
 <link name="base_link">
   <inertial>
-    <origin xyz="-0.009115327490433861 0.00030805565808849657 0.07452875806975676" rpy="0 0 0"/>
-    <mass value="3.833392761738788"/>
-    <inertia ixx="0.016777" iyy="0.029722" izz="0.021198" ixy="1.6e-05" iyz="3.9e-05" ixz="-0.003484"/>
+    <origin xyz="-0.009254800794680978 0.00030186356552978536 0.07136287250840642" rpy="0 0 0"/>
+    <mass value="0.6870543151787526"/>
+    <inertia ixx="0.002614" iyy="0.004939" izz="0.003796" ixy="3e-06" iyz="6e-06" ixz="-0.000506"/>
   </inertial>
   <visual>
     <origin xyz="0 0 0" rpy="0 0 0"/>
     <geometry>
-      <mesh filename="file://$(find Elegoo_to_urdf_description)/meshes/base_link.stl" scale="0.001 0.001 0.001"/>
+      <mesh filename="file://$(find navexbot_description)/meshes/base_link.stl" scale="0.001 0.001 0.001"/>
     </geometry>
     <material name="silver"/>
@@ -20,5 +20,5 @@
     <origin xyz="0 0 0" rpy="0 0 0"/>
     <geometry>
-      <mesh filename="file://$(find Elegoo_to_urdf_description)/meshes/base_link.stl" scale="0.001 0.001 0.001"/>
+      <mesh filename="file://$(find navexbot_description)/meshes/base_link.stl" scale="0.001 0.001 0.001"/>
     </geometry>
   </collision>
@@ -27,11 +27,11 @@
   <inertial>
     <origin xyz="-0.015249901865530185 0.01003722825181954 0.0012500000000014513" rpy="0 0 0"/>
-    <mass value="0.018538509672895963"/>
-    <inertia ixx="2e-06" iyy="3e-06" izz="5e-06" ixy="0.0" iyz="0.0" ixz="0.0"/>
+    <mass value="0.006000809309404922"/>
+    <inertia ixx="1e-06" iyy="1e-06" izz="1e-06" ixy="0.0" iyz="0.0" ixz="-0.0"/>
   </inertial>
   <visual>
     <origin xyz="-0.101915 0.017411 -0.048908" rpy="0 0 0"/>
     <geometry>
-      <mesh filename="file://$(find Elegoo_to_urdf_description)/meshes/Dead_Plate_1.stl" scale="0.001 0.001 0.001"/>
+      <mesh filename="file://$(find navexbot_description)/meshes/Dead_Plate_1.stl" scale="0.001 0.001 0.001"/>
     </geometry>
     <material name="silver"/>
@@ -40,5 +40,5 @@
     <origin xyz="-0.101915 0.017411 -0.048908" rpy="0 0 0"/>
     <geometry>
-      <mesh filename="file://$(find Elegoo_to_urdf_description)/meshes/Dead_Plate_1.stl" scale="0.001 0.001 0.001"/>
+      <mesh filename="file://$(find navexbot_description)/meshes/Dead_Plate_1.stl" scale="0.001 0.001 0.001"/>
     </geometry>
   </collision>
@@ -47,11 +47,11 @@
   <inertial>
     <origin xyz="-0.01419207764726356 -3.2856846282885294e-07 -0.0038831763099285363" rpy="0 0 0"/>
-    <mass value="0.05642275816558916"/>
-    <inertia ixx="4e-06" iyy="6e-06" izz="3e-06" ixy="-0.0" iyz="0.0" ixz="0.0"/>
+    <mass value="0.009861404357094055"/>
+    <inertia ixx="1e-06" iyy="1e-06" izz="1e-06" ixy="-0.0" iyz="0.0" ixz="0.0"/>
   </inertial>
   <visual>
     <origin xyz="-0.100215 -0.001689 -0.051408" rpy="0 0 0"/>
     <geometry>
-      <mesh filename="file://$(find Elegoo_to_urdf_description)/meshes/Servo_1.stl" scale="0.001 0.001 0.001"/>
+      <mesh filename="file://$(find navexbot_description)/meshes/Servo_1.stl" scale="0.001 0.001 0.001"/>
     </geometry>
     <material name="silver"/>
@@ -60,5 +60,5 @@
     <origin xyz="-0.100215 -0.001689 -0.051408" rpy="0 0 0"/>
     <geometry>
-      <mesh filename="file://$(find Elegoo_to_urdf_description)/meshes/Servo_1.stl" scale="0.001 0.001 0.001"/>
+      <mesh filename="file://$(find navexbot_description)/meshes/Servo_1.stl" scale="0.001 0.001 0.001"/>
     </geometry>
   </collision>
@@ -67,11 +67,11 @@
   <inertial>
     <origin xyz="0.0048744154488705865 -3.285684765947511e-07 0.015150516120221058" rpy="0 0 0"/>
-    <mass value="0.027799828090996286"/>
-    <inertia ixx="9e-06" iyy="4e-06" izz="5e-06" ixy="-0.0" iyz="0.0" ixz="-0.0"/>
+    <mass value="0.006020344936903655"/>
+    <inertia ixx="2e-06" iyy="1e-06" izz="1e-06" ixy="-0.0" iyz="0.0" ixz="-0.0"/>
   </inertial>
   <visual>
     <origin xyz="-0.08059 -0.001689 -0.065018" rpy="0 0 0"/>
     <geometry>
-      <mesh filename="file://$(find Elegoo_to_urdf_description)/meshes/Sensor_Mount_Bracket_1.stl" scale="0.001 0.001 0.001"/>
+      <mesh filename="file://$(find navexbot_description)/meshes/Sensor_Mount_Bracket_1.stl" scale="0.001 0.001 0.001"/>
     </geometry>
     <material name="silver"/>
@@ -80,5 +80,5 @@
     <origin xyz="-0.08059 -0.001689 -0.065018" rpy="0 0 0"/>
     <geometry>
-      <mesh filename="file://$(find Elegoo_to_urdf_description)/meshes/Sensor_Mount_Bracket_1.stl" scale="0.001 0.001 0.001"/>
+      <mesh filename="file://$(find navexbot_description)/meshes/Sensor_Mount_Bracket_1.stl" scale="0.001 0.001 0.001"/>
     </geometry>
   </collision>
@@ -86,12 +86,12 @@
 <link name="Ultrasonic_Sensor_1">
   <inertial>
-    <origin xyz="0.004740381871599211 -0.020350330938488658 -0.008123162822331054" rpy="0 0 0"/>
-    <mass value="0.03725196860961161"/>
-    <inertia ixx="7e-06" iyy="1e-06" izz="7e-06" ixy="-0.0" iyz="-0.0" ixz="-0.0"/>
+    <origin xyz="0.004740381707849045 -0.020350330982211375 -0.008123162994376487" rpy="0 0 0"/>
+    <mass value="0.011000008480470561"/>
+    <inertia ixx="2e-06" iyy="0.0" izz="2e-06" ixy="-0.0" iyz="-0.0" ixz="-0.0"/>
   </inertial>
   <visual>
     <origin xyz="-0.08959 -0.022039 -0.094368" rpy="0 0 0"/>
     <geometry>
-      <mesh filename="file://$(find Elegoo_to_urdf_description)/meshes/Ultrasonic_Sensor_1.stl" scale="0.001 0.001 0.001"/>
+      <mesh filename="file://$(find navexbot_description)/meshes/Ultrasonic_Sensor_1.stl" scale="0.001 0.001 0.001"/>
     </geometry>
     <material name="silver"/>
@@ -100,5 +100,185 @@
     <origin xyz="-0.08959 -0.022039 -0.094368" rpy="0 0 0"/>
     <geometry>
-      <mesh filename="file://$(find Elegoo_to_urdf_description)/meshes/Ultrasonic_Sensor_1.stl" scale="0.001 0.001 0.001"/>
+      <mesh filename="file://$(find navexbot_description)/meshes/Ultrasonic_Sensor_1.stl" scale="0.001 0.001 0.001"/>
+    </geometry>
+  </collision>
+</link>
+<link name="Power_Bank_v1_1">
+  <inertial>
+    <origin xyz="0.3969137120101962 -0.26660239809159086 -0.5245509872358798" rpy="0 0 0"/>
+    <mass value="0.5000878365425062"/>
+    <inertia ixx="0.000613" iyy="0.000213" izz="0.000743" ixy="0.0" iyz="0.0" ixz="0.0"/>
+  </inertial>
+  <visual>
+    <origin xyz="0.44 -0.266614 -0.653459" rpy="0 0 0"/>
+    <geometry>
+      <mesh filename="file://$(find navexbot_description)/meshes/Power_Bank_v1_1.stl" scale="0.001 0.001 0.001"/>
+    </geometry>
+    <material name="silver"/>
+  </visual>
+  <collision>
+    <origin xyz="0.44 -0.266614 -0.653459" rpy="0 0 0"/>
+    <geometry>
+      <mesh filename="file://$(find navexbot_description)/meshes/Power_Bank_v1_1.stl" scale="0.001 0.001 0.001"/>
+    </geometry>
+  </collision>
+</link>
+<link name="RASPBERRY_PI_5_1_v1_1">
+  <inertial>
+    <origin xyz="-0.024667496420228745 -0.05471353923003691 0.0053205519092848486" rpy="0 0 0"/>
+    <mass value="0.07999938290722161"/>
+    <inertia ixx="5.3e-05" iyy="2.3e-05" izz="7.2e-05" ixy="-1e-06" iyz="6e-06" ixz="-0.0"/>
+  </inertial>
+  <visual>
+    <origin xyz="-0.069576 -0.039064 -0.112908" rpy="0 0 0"/>
+    <geometry>
+      <mesh filename="file://$(find navexbot_description)/meshes/RASPBERRY_PI_5_1_v1_1.stl" scale="0.001 0.001 0.001"/>
+    </geometry>
+    <material name="silver"/>
+  </visual>
+  <collision>
+    <origin xyz="-0.069576 -0.039064 -0.112908" rpy="0 0 0"/>
+    <geometry>
+      <mesh filename="file://$(find navexbot_description)/meshes/RASPBERRY_PI_5_1_v1_1.stl" scale="0.001 0.001 0.001"/>
+    </geometry>
+  </collision>
+</link>
+<link name="Line_Tracking_Module_1">
+  <inertial>
+    <origin xyz="0.5540313035972204 -0.42631351135466095 -0.5444658120038782" rpy="0 0 0"/>
+    <mass value="0.011999979009967758"/>
+    <inertia ixx="2e-06" iyy="1e-06" izz="3e-06" ixy="-0.0" iyz="0.0" ixz="0.0"/>
+  </inertial>
+  <visual>
+    <origin xyz="0.460696 -0.427264 -0.542551" rpy="0 0 0"/>
+    <geometry>
+      <mesh filename="file://$(find navexbot_description)/meshes/Line_Tracking_Module_1.stl" scale="0.001 0.001 0.001"/>
+    </geometry>
+    <material name="silver"/>
+  </visual>
+  <collision>
+    <origin xyz="0.460696 -0.427264 -0.542551" rpy="0 0 0"/>
+    <geometry>
+      <mesh filename="file://$(find navexbot_description)/meshes/Line_Tracking_Module_1.stl" scale="0.001 0.001 0.001"/>
+    </geometry>
+  </collision>
+</link>
+<link name="Arduino_Mega_v1_1">
+  <inertial>
+    <origin xyz="-0.024846623231800355 0.029164935620271216 0.0028012635578156322" rpy="0 0 0"/>
+    <mass value="0.03699959187591492"/>
+    <inertia ixx="4.2e-05" iyy="1e-05" izz="5.1e-05" ixy="-1e-06" iyz="1e-06" ixz="0.0"/>
+  </inertial>
+  <visual>
+    <origin xyz="-0.021607 0.036831 -0.048908" rpy="0 0 0"/>
+    <geometry>
+      <mesh filename="file://$(find navexbot_description)/meshes/Arduino_Mega_v1_1.stl" scale="0.001 0.001 0.001"/>
+    </geometry>
+    <material name="silver"/>
+  </visual>
+  <collision>
+    <origin xyz="-0.021607 0.036831 -0.048908" rpy="0 0 0"/>
+    <geometry>
+      <mesh filename="file://$(find navexbot_description)/meshes/Arduino_Mega_v1_1.stl" scale="0.001 0.001 0.001"/>
+    </geometry>
+  </collision>
+</link>
+<link name="Expansion_Board_1">
+  <inertial>
+    <origin xyz="-0.08726576052727084 0.08646332521308203 -0.0034230357875419254" rpy="0 0 0"/>
+    <mass value="0.01901859698907641"/>
+    <inertia ixx="6e-06" iyy="5e-06" izz="1e-05" ixy="0.0" iyz="0.0" ixz="-0.0"/>
+  </inertial>
+  <visual>
+    <origin xyz="-0.083115 0.078424 -0.065747" rpy="0 0 0"/>
+    <geometry>
+      <mesh filename="file://$(find navexbot_description)/meshes/Expansion_Board_1.stl" scale="0.001 0.001 0.001"/>
+    </geometry>
+    <material name="silver"/>
+  </visual>
+  <collision>
+    <origin xyz="-0.083115 0.078424 -0.065747" rpy="0 0 0"/>
+    <geometry>
+      <mesh filename="file://$(find navexbot_description)/meshes/Expansion_Board_1.stl" scale="0.001 0.001 0.001"/>
+    </geometry>
+  </collision>
+</link>
+<link name="wheel_1_1">
+  <inertial>
+    <origin xyz="0.4327751903063669 -0.4281664221543372 -0.5405508438975558" rpy="0 0 0"/>
+    <mass value="0.037002404972170014"/>
+    <inertia ixx="1.5e-05" iyy="2.5e-05" izz="1.5e-05" ixy="-0.0" iyz="-0.0" ixz="0.0"/>
+  </inertial>
+  <visual>
+    <origin xyz="0.393843 -0.36047 -0.558301" rpy="0 0 0"/>
+    <geometry>
+      <mesh filename="file://$(find navexbot_description)/meshes/wheel_1_1.stl" scale="0.001 0.001 0.001"/>
+    </geometry>
+    <material name="silver"/>
+  </visual>
+  <collision>
+    <origin xyz="0.393843 -0.36047 -0.558301" rpy="0 0 0"/>
+    <geometry>
+      <mesh filename="file://$(find navexbot_description)/meshes/wheel_1_1.stl" scale="0.001 0.001 0.001"/>
+    </geometry>
+  </collision>
+</link>
+<link name="wheel_4_1">
+  <inertial>
+    <origin xyz="0.5258811943895968 -0.2918523043337162 -0.5405508379440966" rpy="0 0 0"/>
+    <mass value="0.03700242493307289"/>
+    <inertia ixx="1.5e-05" iyy="2.5e-05" izz="1.5e-05" ixy="0.0" iyz="-0.0" ixz="0.0"/>
+  </inertial>
+  <visual>
+    <origin xyz="0.486949 -0.36047 -0.558301" rpy="0 0 0"/>
+    <geometry>
+      <mesh filename="file://$(find navexbot_description)/meshes/wheel_4_1.stl" scale="0.001 0.001 0.001"/>
+    </geometry>
+    <material name="silver"/>
+  </visual>
+  <collision>
+    <origin xyz="0.486949 -0.36047 -0.558301" rpy="0 0 0"/>
+    <geometry>
+      <mesh filename="file://$(find navexbot_description)/meshes/wheel_4_1.stl" scale="0.001 0.001 0.001"/>
+    </geometry>
+  </collision>
+</link>
+<link name="wheel_3_1">
+  <inertial>
+    <origin xyz="0.44394981714587184 -0.2099212285643192 -0.5405509961025838" rpy="0 0 0"/>
+    <mass value="0.03700242493307289"/>
+    <inertia ixx="1.5e-05" iyy="2.5e-05" izz="1.5e-05" ixy="0.0" iyz="-0.0" ixz="0.0"/>
+  </inertial>
+  <visual>
+    <origin xyz="0.486949 -0.278539 -0.558301" rpy="0 0 0"/>
+    <geometry>
+      <mesh filename="file://$(find navexbot_description)/meshes/wheel_3_1.stl" scale="0.001 0.001 0.001"/>
+    </geometry>
+    <material name="silver"/>
+  </visual>
+  <collision>
+    <origin xyz="0.486949 -0.278539 -0.558301" rpy="0 0 0"/>
+    <geometry>
+      <mesh filename="file://$(find navexbot_description)/meshes/wheel_3_1.stl" scale="0.001 0.001 0.001"/>
+    </geometry>
+  </collision>
+</link>
+<link name="wheel_2_1">
+  <inertial>
+    <origin xyz="0.35084381306264295 -0.34623549792373326 -0.5405510020560437" rpy="0 0 0"/>
+    <mass value="0.037002404972170014"/>
+    <inertia ixx="1.5e-05" iyy="2.5e-05" izz="1.5e-05" ixy="-0.0" iyz="-0.0" ixz="0.0"/>
+  </inertial>
+  <visual>
+    <origin xyz="0.393843 -0.278539 -0.558301" rpy="0 0 0"/>
+    <geometry>
+      <mesh filename="file://$(find navexbot_description)/meshes/wheel_2_1.stl" scale="0.001 0.001 0.001"/>
+    </geometry>
+    <material name="silver"/>
+  </visual>
+  <collision>
+    <origin xyz="0.393843 -0.278539 -0.558301" rpy="0 0 0"/>
+    <geometry>
+      <mesh filename="file://$(find navexbot_description)/meshes/wheel_2_1.stl" scale="0.001 0.001 0.001"/>
     </geometry>
   </collision>
@@ -106,199 +286,19 @@
 <link name="C1M1_appearance_V2_20230926.3d_model_v2_1">
   <inertial>
-    <origin xyz="8.370960599731608e-05 -9.423957307502595e-05 0.01399453162565878" rpy="0 0 0"/>
-    <mass value="0.25439238942428605"/>
-    <inertia ixx="0.000111" iyy="0.000111" izz="0.000157" ixy="-0.0" iyz="-0.0" ixz="0.0"/>
-  </inertial>
-  <visual>
-    <origin xyz="-0.045076 -6.4e-05 -0.176908" rpy="0 0 0"/>
-    <geometry>
-      <mesh filename="file://$(find Elegoo_to_urdf_description)/meshes/C1M1_appearance_V2_20230926.3d_model_v2_1.stl" scale="0.001 0.001 0.001"/>
-    </geometry>
-    <material name="silver"/>
-  </visual>
-  <collision>
-    <origin xyz="-0.045076 -6.4e-05 -0.176908" rpy="0 0 0"/>
-    <geometry>
-      <mesh filename="file://$(find Elegoo_to_urdf_description)/meshes/C1M1_appearance_V2_20230926.3d_model_v2_1.stl" scale="0.001 0.001 0.001"/>
-    </geometry>
-  </collision>
-</link>
-<link name="Power_Bank_v1_1">
-  <inertial>
-    <origin xyz="0.3969137120101962 -0.26660239809159086 -0.5245509872358798" rpy="0 0 0"/>
-    <mass value="1.9212497023729622"/>
-    <inertia ixx="0.002353" iyy="0.000817" izz="0.002853" ixy="0.0" iyz="0.0" ixz="0.0"/>
-  </inertial>
-  <visual>
-    <origin xyz="0.44 -0.266614 -0.653459" rpy="0 0 0"/>
-    <geometry>
-      <mesh filename="file://$(find Elegoo_to_urdf_description)/meshes/Power_Bank_v1_1.stl" scale="0.001 0.001 0.001"/>
-    </geometry>
-    <material name="silver"/>
-  </visual>
-  <collision>
-    <origin xyz="0.44 -0.266614 -0.653459" rpy="0 0 0"/>
-    <geometry>
-      <mesh filename="file://$(find Elegoo_to_urdf_description)/meshes/Power_Bank_v1_1.stl" scale="0.001 0.001 0.001"/>
-    </geometry>
-  </collision>
-</link>
-<link name="RASPBERRY_PI_5_1_v1_1">
-  <inertial>
-    <origin xyz="-0.024667479251557496 -0.05471357115382812 0.005320553085662497" rpy="0 0 0"/>
-    <mass value="0.1407428995912446"/>
-    <inertia ixx="9.4e-05" iyy="4.1e-05" izz="0.000127" ixy="-1e-06" iyz="1e-05" ixz="-0.0"/>
-  </inertial>
-  <visual>
-    <origin xyz="-0.069576 -0.039064 -0.112908" rpy="0 0 0"/>
-    <geometry>
-      <mesh filename="file://$(find Elegoo_to_urdf_description)/meshes/RASPBERRY_PI_5_1_v1_1.stl" scale="0.001 0.001 0.001"/>
-    </geometry>
-    <material name="silver"/>
-  </visual>
-  <collision>
-    <origin xyz="-0.069576 -0.039064 -0.112908" rpy="0 0 0"/>
-    <geometry>
-      <mesh filename="file://$(find Elegoo_to_urdf_description)/meshes/RASPBERRY_PI_5_1_v1_1.stl" scale="0.001 0.001 0.001"/>
-    </geometry>
-  </collision>
-</link>
-<link name="Line_Tracking_Module_1">
-  <inertial>
-    <origin xyz="0.5540313035972204 -0.42631351135466095 -0.5444658120038782" rpy="0 0 0"/>
-    <mass value="0.022807020126442847"/>
-    <inertia ixx="4e-06" iyy="2e-06" izz="5e-06" ixy="-0.0" iyz="0.0" ixz="0.0"/>
-  </inertial>
-  <visual>
-    <origin xyz="0.460696 -0.427264 -0.542551" rpy="0 0 0"/>
-    <geometry>
-      <mesh filename="file://$(find Elegoo_to_urdf_description)/meshes/Line_Tracking_Module_1.stl" scale="0.001 0.001 0.001"/>
-    </geometry>
-    <material name="silver"/>
-  </visual>
-  <collision>
-    <origin xyz="0.460696 -0.427264 -0.542551" rpy="0 0 0"/>
-    <geometry>
-      <mesh filename="file://$(find Elegoo_to_urdf_description)/meshes/Line_Tracking_Module_1.stl" scale="0.001 0.001 0.001"/>
-    </geometry>
-  </collision>
-</link>
-<link name="Arduino_Mega_v1_1">
-  <inertial>
-    <origin xyz="-0.024846623231800355 0.029164935620271216 0.0028012635578156322" rpy="0 0 0"/>
-    <mass value="0.11616477871692679"/>
-    <inertia ixx="0.00013" iyy="3.1e-05" izz="0.000159" ixy="-3e-06" iyz="3e-06" ixz="0.0"/>
-  </inertial>
-  <visual>
-    <origin xyz="-0.021607 0.036831 -0.048908" rpy="0 0 0"/>
-    <geometry>
-      <mesh filename="file://$(find Elegoo_to_urdf_description)/meshes/Arduino_Mega_v1_1.stl" scale="0.001 0.001 0.001"/>
-    </geometry>
-    <material name="silver"/>
-  </visual>
-  <collision>
-    <origin xyz="-0.021607 0.036831 -0.048908" rpy="0 0 0"/>
-    <geometry>
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