Commit message: feat(urdf): add color materials to robot components

File: navexbot_description/urdf/materials.xacro (robot description, xacro)
@@ -1,6 +1,24 @@
 <?xml version="1.0" ?>
-<robot name="Elegoo_to_urdf" xmlns:xacro="http://www.ros.org/wiki/xacro" >
+<robot name="navexbot" xmlns:xacro="http://www.ros.org/wiki/xacro" >
 <material name="silver">
   <color rgba="0.700 0.700 0.700 1.000"/>
 </material>
+<material name="black">
+  <color rgba="0.000 0.000 0.000 1.000"/>
+</material>
+<material name="blue">
+  <color rgba="0.043 0.651 0.875 1.000"/>
+</material>
+<material name="yellow">
+  <color rgba="1.000 1.000 0.000 1.000"/>
+</material>
+<material name="sage">
+  <color rgba="0.518 0.600 0.310 1.000"/>
+</material>
+<material name="teal">
+  <color rgba="0.000 0.500 0.500 1.000"/>
+</material>
+<material name="green">
+  <color rgba="0.388 0.639 0.380 1.000"/>
+</material>
 </robot>

File: navexbot_description/urdf/navexbot.xacro (robot description, xacro)
@@ -1,7 +1,7 @@
 <?xml version="1.0" ?>
-<robot name="Elegoo_to_urdf" xmlns:xacro="http://www.ros.org/wiki/xacro">
-<xacro:include filename="$(find Elegoo_to_urdf_description)/urdf/materials.xacro" />
-<xacro:include filename="$(find Elegoo_to_urdf_description)/urdf/Elegoo_to_urdf.trans" />
-<xacro:include filename="$(find Elegoo_to_urdf_description)/urdf/Elegoo_to_urdf.gazebo" />
+<robot name="navexbot" xmlns:xacro="http://www.ros.org/wiki/xacro">
+<xacro:include filename="$(find navexbot_description)/urdf/materials.xacro" />
+<xacro:include filename="$(find navexbot_description)/urdf/navexbot.trans" />
+<xacro:include filename="$(find navexbot_description)/urdf/navexbot.gazebo" />
 <link name="base_link">
   <inertial>
@@ -13,12 +13,12 @@
     <origin xyz="0 0 0" rpy="0 0 0"/>
     <geometry>
-      <mesh filename="file://$(find Elegoo_to_urdf_description)/meshes/base_link.stl" scale="0.001 0.001 0.001"/>
-    </geometry>
-    <material name="silver"/>
+      <mesh filename="file://$(find navexbot_description)/meshes/base_link.stl" scale="0.001 0.001 0.001"/>
+    </geometry>
+    <material name="black"/>
   </visual>
   <collision>
     <origin xyz="0 0 0" rpy="0 0 0"/>
     <geometry>
-      <mesh filename="file://$(find Elegoo_to_urdf_description)/meshes/base_link.stl" scale="0.001 0.001 0.001"/>
+      <mesh filename="file://$(find navexbot_description)/meshes/base_link.stl" scale="0.001 0.001 0.001"/>
     </geometry>
   </collision>
@@ -33,12 +33,12 @@
     <origin xyz="-0.101915 0.017411 -0.048908" rpy="0 0 0"/>
     <geometry>
-      <mesh filename="file://$(find Elegoo_to_urdf_description)/meshes/Dead_Plate_1.stl" scale="0.001 0.001 0.001"/>
-    </geometry>
-    <material name="silver"/>
+      <mesh filename="file://$(find navexbot_description)/meshes/Dead_Plate_1.stl" scale="0.001 0.001 0.001"/>
+    </geometry>
+    <material name="black"/>
   </visual>
   <collision>
     <origin xyz="-0.101915 0.017411 -0.048908" rpy="0 0 0"/>
     <geometry>
-      <mesh filename="file://$(find Elegoo_to_urdf_description)/meshes/Dead_Plate_1.stl" scale="0.001 0.001 0.001"/>
+      <mesh filename="file://$(find navexbot_description)/meshes/Dead_Plate_1.stl" scale="0.001 0.001 0.001"/>
     </geometry>
   </collision>
@@ -53,12 +53,12 @@
     <origin xyz="-0.100215 -0.001689 -0.051408" rpy="0 0 0"/>
     <geometry>
-      <mesh filename="file://$(find Elegoo_to_urdf_description)/meshes/Servo_1.stl" scale="0.001 0.001 0.001"/>
-    </geometry>
-    <material name="silver"/>
+      <mesh filename="file://$(find navexbot_description)/meshes/Servo_1.stl" scale="0.001 0.001 0.001"/>
+    </geometry>
+    <material name="blue"/>
   </visual>
   <collision>
     <origin xyz="-0.100215 -0.001689 -0.051408" rpy="0 0 0"/>
     <geometry>
-      <mesh filename="file://$(find Elegoo_to_urdf_description)/meshes/Servo_1.stl" scale="0.001 0.001 0.001"/>
+      <mesh filename="file://$(find navexbot_description)/meshes/Servo_1.stl" scale="0.001 0.001 0.001"/>
     </geometry>
   </collision>
@@ -73,12 +73,12 @@
     <origin xyz="-0.08059 -0.001689 -0.065018" rpy="0 0 0"/>
     <geometry>
-      <mesh filename="file://$(find Elegoo_to_urdf_description)/meshes/Sensor_Mount_Bracket_1.stl" scale="0.001 0.001 0.001"/>
-    </geometry>
-    <material name="silver"/>
+      <mesh filename="file://$(find navexbot_description)/meshes/Sensor_Mount_Bracket_1.stl" scale="0.001 0.001 0.001"/>
+    </geometry>
+    <material name="black"/>
   </visual>
   <collision>
     <origin xyz="-0.08059 -0.001689 -0.065018" rpy="0 0 0"/>
     <geometry>
-      <mesh filename="file://$(find Elegoo_to_urdf_description)/meshes/Sensor_Mount_Bracket_1.stl" scale="0.001 0.001 0.001"/>
+      <mesh filename="file://$(find navexbot_description)/meshes/Sensor_Mount_Bracket_1.stl" scale="0.001 0.001 0.001"/>
     </geometry>
   </collision>
@@ -93,5 +93,5 @@
     <origin xyz="-0.08959 -0.022039 -0.094368" rpy="0 0 0"/>
     <geometry>
-      <mesh filename="file://$(find Elegoo_to_urdf_description)/meshes/Ultrasonic_Sensor_1.stl" scale="0.001 0.001 0.001"/>
+      <mesh filename="file://$(find navexbot_description)/meshes/Ultrasonic_Sensor_1.stl" scale="0.001 0.001 0.001"/>
     </geometry>
     <material name="silver"/>
@@ -100,5 +100,5 @@
     <origin xyz="-0.08959 -0.022039 -0.094368" rpy="0 0 0"/>
     <geometry>
-      <mesh filename="file://$(find Elegoo_to_urdf_description)/meshes/Ultrasonic_Sensor_1.stl" scale="0.001 0.001 0.001"/>
+      <mesh filename="file://$(find navexbot_description)/meshes/Ultrasonic_Sensor_1.stl" scale="0.001 0.001 0.001"/>
     </geometry>
   </collision>
@@ -113,12 +113,12 @@
     <origin xyz="-0.045076 -6.4e-05 -0.176908" rpy="0 0 0"/>
     <geometry>
-      <mesh filename="file://$(find Elegoo_to_urdf_description)/meshes/C1M1_appearance_V2_20230926.3d_model_v2_1.stl" scale="0.001 0.001 0.001"/>
-    </geometry>
-    <material name="silver"/>
+      <mesh filename="file://$(find navexbot_description)/meshes/C1M1_appearance_V2_20230926.3d_model_v2_1.stl" scale="0.001 0.001 0.001"/>
+    </geometry>
+    <material name="blue"/>
   </visual>
   <collision>
     <origin xyz="-0.045076 -6.4e-05 -0.176908" rpy="0 0 0"/>
     <geometry>
-      <mesh filename="file://$(find Elegoo_to_urdf_description)/meshes/C1M1_appearance_V2_20230926.3d_model_v2_1.stl" scale="0.001 0.001 0.001"/>
+      <mesh filename="file://$(find navexbot_description)/meshes/C1M1_appearance_V2_20230926.3d_model_v2_1.stl" scale="0.001 0.001 0.001"/>
     </geometry>
   </collision>
@@ -133,12 +133,12 @@
     <origin xyz="0.44 -0.266614 -0.653459" rpy="0 0 0"/>
     <geometry>
-      <mesh filename="file://$(find Elegoo_to_urdf_description)/meshes/Power_Bank_v1_1.stl" scale="0.001 0.001 0.001"/>
-    </geometry>
-    <material name="silver"/>
+      <mesh filename="file://$(find navexbot_description)/meshes/Power_Bank_v1_1.stl" scale="0.001 0.001 0.001"/>
+    </geometry>
+    <material name="sage"/>
   </visual>
   <collision>
     <origin xyz="0.44 -0.266614 -0.653459" rpy="0 0 0"/>
     <geometry>
-      <mesh filename="file://$(find Elegoo_to_urdf_description)/meshes/Power_Bank_v1_1.stl" scale="0.001 0.001 0.001"/>
+      <mesh filename="file://$(find navexbot_description)/meshes/Power_Bank_v1_1.stl" scale="0.001 0.001 0.001"/>
     </geometry>
   </collision>
@@ -153,12 +153,12 @@
     <origin xyz="-0.069576 -0.039064 -0.112908" rpy="0 0 0"/>
     <geometry>
-      <mesh filename="file://$(find Elegoo_to_urdf_description)/meshes/RASPBERRY_PI_5_1_v1_1.stl" scale="0.001 0.001 0.001"/>
-    </geometry>
-    <material name="silver"/>
+      <mesh filename="file://$(find navexbot_description)/meshes/RASPBERRY_PI_5_1_v1_1.stl" scale="0.001 0.001 0.001"/>
+    </geometry>
+    <material name="green"/>
   </visual>
   <collision>
     <origin xyz="-0.069576 -0.039064 -0.112908" rpy="0 0 0"/>
     <geometry>
-      <mesh filename="file://$(find Elegoo_to_urdf_description)/meshes/RASPBERRY_PI_5_1_v1_1.stl" scale="0.001 0.001 0.001"/>
+      <mesh filename="file://$(find navexbot_description)/meshes/RASPBERRY_PI_5_1_v1_1.stl" scale="0.001 0.001 0.001"/>
     </geometry>
   </collision>
@@ -173,5 +173,5 @@
     <origin xyz="0.460696 -0.427264 -0.542551" rpy="0 0 0"/>
     <geometry>
-      <mesh filename="file://$(find Elegoo_to_urdf_description)/meshes/Line_Tracking_Module_1.stl" scale="0.001 0.001 0.001"/>
+      <mesh filename="file://$(find navexbot_description)/meshes/Line_Tracking_Module_1.stl" scale="0.001 0.001 0.001"/>
     </geometry>
     <material name="silver"/>
@@ -180,5 +180,5 @@
     <origin xyz="0.460696 -0.427264 -0.542551" rpy="0 0 0"/>
     <geometry>
-      <mesh filename="file://$(find Elegoo_to_urdf_description)/meshes/Line_Tracking_Module_1.stl" scale="0.001 0.001 0.001"/>
+      <mesh filename="file://$(find navexbot_description)/meshes/Line_Tracking_Module_1.stl" scale="0.001 0.001 0.001"/>
     </geometry>
   </collision>
@@ -193,12 +193,12 @@
     <origin xyz="-0.021607 0.036831 -0.048908" rpy="0 0 0"/>
     <geometry>
-      <mesh filename="file://$(find Elegoo_to_urdf_description)/meshes/Arduino_Mega_v1_1.stl" scale="0.001 0.001 0.001"/>
-    </geometry>
-    <material name="silver"/>
+      <mesh filename="file://$(find navexbot_description)/meshes/Arduino_Mega_v1_1.stl" scale="0.001 0.001 0.001"/>
+    </geometry>
+    <material name="teal"/>
   </visual>
   <collision>
     <origin xyz="-0.021607 0.036831 -0.048908" rpy="0 0 0"/>
     <geometry>
-      <mesh filename="file://$(find Elegoo_to_urdf_description)/meshes/Arduino_Mega_v1_1.stl" scale="0.001 0.001 0.001"/>
+      <mesh filename="file://$(find navexbot_description)/meshes/Arduino_Mega_v1_1.stl" scale="0.001 0.001 0.001"/>
     </geometry>
   </collision>
@@ -213,12 +213,12 @@
     <origin xyz="-0.083115 0.078424 -0.065747" rpy="0 0 0"/>
     <geometry>
-      <mesh filename="file://$(find Elegoo_to_urdf_description)/meshes/Expansion_Board_1.stl" scale="0.001 0.001 0.001"/>
-    </geometry>
-    <material name="silver"/>
+      <mesh filename="file://$(find navexbot_description)/meshes/Expansion_Board_1.stl" scale="0.001 0.001 0.001"/>
+    </geometry>
+    <material name="black"/>
   </visual>
   <collision>
     <origin xyz="-0.083115 0.078424 -0.065747" rpy="0 0 0"/>
     <geometry>
-      <mesh filename="file://$(find Elegoo_to_urdf_description)/meshes/Expansion_Board_1.stl" scale="0.001 0.001 0.001"/>
+      <mesh filename="file://$(find navexbot_description)/meshes/Expansion_Board_1.stl" scale="0.001 0.001 0.001"/>
     </geometry>
   </collision>
@@ -233,12 +233,12 @@
     <origin xyz="0.393843 -0.36047 -0.558301" rpy="0 0 0"/>
     <geometry>
-      <mesh filename="file://$(find Elegoo_to_urdf_description)/meshes/wheel_1_1.stl" scale="0.001 0.001 0.001"/>
-    </geometry>
-    <material name="silver"/>
+      <mesh filename="file://$(find navexbot_description)/meshes/wheel_1_1.stl" scale="0.001 0.001 0.001"/>
+    </geometry>
+    <material name="yellow"/>
   </visual>
   <collision>
     <origin xyz="0.393843 -0.36047 -0.558301" rpy="0 0 0"/>
     <geometry>
-      <mesh filename="file://$(find Elegoo_to_urdf_description)/meshes/wheel_1_1.stl" scale="0.001 0.001 0.001"/>
+      <mesh filename="file://$(find navexbot_description)/meshes/wheel_1_1.stl" scale="0.001 0.001 0.001"/>
     </geometry>
   </collision>
@@ -253,12 +253,12 @@
     <origin xyz="0.486949 -0.36047 -0.558301" rpy="0 0 0"/>
     <geometry>
-      <mesh filename="file://$(find Elegoo_to_urdf_description)/meshes/wheel_4_1.stl" scale="0.001 0.001 0.001"/>
-    </geometry>
-    <material name="silver"/>
+      <mesh filename="file://$(find navexbot_description)/meshes/wheel_4_1.stl" scale="0.001 0.001 0.001"/>
+    </geometry>
+    <material name="yellow"/>
   </visual>
   <collision>
     <origin xyz="0.486949 -0.36047 -0.558301" rpy="0 0 0"/>
     <geometry>
-      <mesh filename="file://$(find Elegoo_to_urdf_description)/meshes/wheel_4_1.stl" scale="0.001 0.001 0.001"/>
+      <mesh filename="file://$(find navexbot_description)/meshes/wheel_4_1.stl" scale="0.001 0.001 0.001"/>
     </geometry>
   </collision>
@@ -273,12 +273,12 @@
     <origin xyz="0.486949 -0.278539 -0.558301" rpy="0 0 0"/>
     <geometry>
-      <mesh filename="file://$(find Elegoo_to_urdf_description)/meshes/wheel_3_1.stl" scale="0.001 0.001 0.001"/>
-    </geometry>
-    <material name="silver"/>
+      <mesh filename="file://$(find navexbot_description)/meshes/wheel_3_1.stl" scale="0.001 0.001 0.001"/>
+    </geometry>
+    <material name="yellow"/>
   </visual>
   <collision>
     <origin xyz="0.486949 -0.278539 -0.558301" rpy="0 0 0"/>
     <geometry>
-      <mesh filename="file://$(find Elegoo_to_urdf_description)/meshes/wheel_3_1.stl" scale="0.001 0.001 0.001"/>
+      <mesh filename="file://$(find navexbot_description)/meshes/wheel_3_1.stl" scale="0.001 0.001 0.001"/>
     </geometry>
   </collision>
@@ -293,12 +293,12 @@
     <origin xyz="0.393843 -0.278539 -0.558301" rpy="0 0 0"/>
     <geometry>
-      <mesh filename="file://$(find Elegoo_to_urdf_description)/meshes/wheel_2_1.stl" scale="0.001 0.001 0.001"/>
-    </geometry>
-    <material name="silver"/>
+      <mesh filename="file://$(find navexbot_description)/meshes/wheel_2_1.stl" scale="0.001 0.001 0.001"/>
+    </geometry>
+    <material name="yellow"/>
   </visual>
   <collision>
     <origin xyz="0.393843 -0.278539 -0.558301" rpy="0 0 0"/>
     <geometry>
-      <mesh filename="file://$(find Elegoo_to_urdf_description)/meshes/wheel_2_1.stl" scale="0.001 0.001 0.001"/>
+      <mesh filename="file://$(find navexbot_description)/meshes/wheel_2_1.stl" scale="0.001 0.001 0.001"/>
     </geometry>
   </collision>
