Commit message: [fix] reposition origin for all components

File: navexbot_description/urdf/materials.xacro (robot description, xacro)
@@ -4,21 +4,3 @@
   <color rgba="0.700 0.700 0.700 1.000"/>
 </material>
-<material name="black">
-  <color rgba="0.000 0.000 0.000 1.000"/>
-</material>
-<material name="blue">
-  <color rgba="0.043 0.651 0.875 1.000"/>
-</material>
-<material name="yellow">
-  <color rgba="1.000 1.000 0.000 1.000"/>
-</material>
-<material name="sage">
-  <color rgba="0.518 0.600 0.310 1.000"/>
-</material>
-<material name="teal">
-  <color rgba="0.000 0.500 0.500 1.000"/>
-</material>
-<material name="green">
-  <color rgba="0.388 0.639 0.380 1.000"/>
-</material>
 </robot>

File: navexbot_description/urdf/navexbot.xacro (robot description, xacro)
@@ -6,6 +6,6 @@
 <link name="base_link">
   <inertial>
-    <origin xyz="-0.009254800794680978 0.00030186356552978536 0.07136287250840642" rpy="0 0 0"/>
-    <mass value="0.6870543151787526"/>
+    <origin xyz="0.3138020472259591 0.707742333605108 0.651058897421196" rpy="0 0 0"/>
+    <mass value="0.6870544631870525"/>
     <inertia ixx="0.002614" iyy="0.004939" izz="0.003796" ixy="3e-06" iyz="6e-06" ixz="-0.000506"/>
   </inertial>
@@ -24,121 +24,81 @@
   </collision>
 </link>
-<link name="Dead_Plate_1">
-  <inertial>
-    <origin xyz="-0.015249901865530185 0.01003722825181954 0.0012500000000014513" rpy="0 0 0"/>
-    <mass value="0.006000809309404922"/>
-    <inertia ixx="1e-06" iyy="1e-06" izz="1e-06" ixy="0.0" iyz="0.0" ixz="-0.0"/>
-  </inertial>
-  <visual>
-    <origin xyz="-0.101915 0.017411 -0.048908" rpy="0 0 0"/>
-    <geometry>
-      <mesh filename="file://$(find navexbot_description)/meshes/Dead_Plate_1.stl" scale="0.001 0.001 0.001"/>
-    </geometry>
-    <material name="silver"/>
-  </visual>
-  <collision>
-    <origin xyz="-0.101915 0.017411 -0.048908" rpy="0 0 0"/>
-    <geometry>
-      <mesh filename="file://$(find navexbot_description)/meshes/Dead_Plate_1.stl" scale="0.001 0.001 0.001"/>
-    </geometry>
-  </collision>
-</link>
-<link name="Servo_1">
-  <inertial>
-    <origin xyz="-0.01419207764726356 -3.2856846282885294e-07 -0.0038831763099285363" rpy="0 0 0"/>
-    <mass value="0.009861404357094055"/>
-    <inertia ixx="1e-06" iyy="1e-06" izz="1e-06" ixy="-0.0" iyz="0.0" ixz="0.0"/>
-  </inertial>
-  <visual>
-    <origin xyz="-0.100215 -0.001689 -0.051408" rpy="0 0 0"/>
-    <geometry>
-      <mesh filename="file://$(find navexbot_description)/meshes/Servo_1.stl" scale="0.001 0.001 0.001"/>
-    </geometry>
-    <material name="silver"/>
-  </visual>
-  <collision>
-    <origin xyz="-0.100215 -0.001689 -0.051408" rpy="0 0 0"/>
-    <geometry>
-      <mesh filename="file://$(find navexbot_description)/meshes/Servo_1.stl" scale="0.001 0.001 0.001"/>
-    </geometry>
-  </collision>
-</link>
-<link name="Sensor_Mount_Bracket_1">
-  <inertial>
-    <origin xyz="0.0048744154488705865 -3.285684765947511e-07 0.015150516120221058" rpy="0 0 0"/>
-    <mass value="0.006020344936903655"/>
-    <inertia ixx="2e-06" iyy="1e-06" izz="1e-06" ixy="-0.0" iyz="0.0" ixz="-0.0"/>
-  </inertial>
-  <visual>
-    <origin xyz="-0.08059 -0.001689 -0.065018" rpy="0 0 0"/>
-    <geometry>
-      <mesh filename="file://$(find navexbot_description)/meshes/Sensor_Mount_Bracket_1.stl" scale="0.001 0.001 0.001"/>
-    </geometry>
-    <material name="silver"/>
-  </visual>
-  <collision>
-    <origin xyz="-0.08059 -0.001689 -0.065018" rpy="0 0 0"/>
-    <geometry>
-      <mesh filename="file://$(find navexbot_description)/meshes/Sensor_Mount_Bracket_1.stl" scale="0.001 0.001 0.001"/>
-    </geometry>
-  </collision>
-</link>
-<link name="Ultrasonic_Sensor_1">
-  <inertial>
-    <origin xyz="0.004740381707849045 -0.020350330982211375 -0.008123162994376487" rpy="0 0 0"/>
-    <mass value="0.011000008480470561"/>
-    <inertia ixx="2e-06" iyy="0.0" izz="2e-06" ixy="-0.0" iyz="-0.0" ixz="-0.0"/>
-  </inertial>
-  <visual>
-    <origin xyz="-0.08959 -0.022039 -0.094368" rpy="0 0 0"/>
-    <geometry>
-      <mesh filename="file://$(find navexbot_description)/meshes/Ultrasonic_Sensor_1.stl" scale="0.001 0.001 0.001"/>
-    </geometry>
-    <material name="silver"/>
-  </visual>
-  <collision>
-    <origin xyz="-0.08959 -0.022039 -0.094368" rpy="0 0 0"/>
-    <geometry>
-      <mesh filename="file://$(find navexbot_description)/meshes/Ultrasonic_Sensor_1.stl" scale="0.001 0.001 0.001"/>
-    </geometry>
-  </collision>
-</link>
-<link name="Power_Bank_v1_1">
-  <inertial>
-    <origin xyz="0.3969137120101962 -0.26660239809159086 -0.5245509872358798" rpy="0 0 0"/>
-    <mass value="0.5000878365425062"/>
-    <inertia ixx="0.000613" iyy="0.000213" izz="0.000743" ixy="0.0" iyz="0.0" ixz="0.0"/>
-  </inertial>
-  <visual>
-    <origin xyz="0.44 -0.266614 -0.653459" rpy="0 0 0"/>
-    <geometry>
-      <mesh filename="file://$(find navexbot_description)/meshes/Power_Bank_v1_1.stl" scale="0.001 0.001 0.001"/>
-    </geometry>
-    <material name="silver"/>
-  </visual>
-  <collision>
-    <origin xyz="0.44 -0.266614 -0.653459" rpy="0 0 0"/>
-    <geometry>
-      <mesh filename="file://$(find navexbot_description)/meshes/Power_Bank_v1_1.stl" scale="0.001 0.001 0.001"/>
-    </geometry>
-  </collision>
-</link>
-<link name="RASPBERRY_PI_5_1_v1_1">
-  <inertial>
-    <origin xyz="-0.024667496420228745 -0.05471353923003691 0.0053205519092848486" rpy="0 0 0"/>
-    <mass value="0.07999938290722161"/>
-    <inertia ixx="5.3e-05" iyy="2.3e-05" izz="7.2e-05" ixy="-1e-06" iyz="6e-06" ixz="-0.0"/>
-  </inertial>
-  <visual>
-    <origin xyz="-0.069576 -0.039064 -0.112908" rpy="0 0 0"/>
-    <geometry>
-      <mesh filename="file://$(find navexbot_description)/meshes/RASPBERRY_PI_5_1_v1_1.stl" scale="0.001 0.001 0.001"/>
-    </geometry>
-    <material name="silver"/>
-  </visual>
-  <collision>
-    <origin xyz="-0.069576 -0.039064 -0.112908" rpy="0 0 0"/>
-    <geometry>
-      <mesh filename="file://$(find navexbot_description)/meshes/RASPBERRY_PI_5_1_v1_1.stl" scale="0.001 0.001 0.001"/>
+<link name="Wheel_LF_1">
+  <inertial>
+    <origin xyz="-0.3230569549805825 -0.6888368425088942 -0.5816957930037309" rpy="0 0 0"/>
+    <mass value="0.037002439542276624"/>
+    <inertia ixx="1.5e-05" iyy="2.5e-05" izz="1.5e-05" ixy="-0.0" iyz="0.0" ixz="0.0"/>
+  </inertial>
+  <visual>
+    <origin xyz="-0.685046 -1.461895 -1.179142" rpy="0 0 0"/>
+    <geometry>
+      <mesh filename="file://$(find navexbot_description)/meshes/Wheel_LF_1.stl" scale="0.001 0.001 0.001"/>
+    </geometry>
+    <material name="silver"/>
+  </visual>
+  <collision>
+    <origin xyz="-0.685046 -1.461895 -1.179142" rpy="0 0 0"/>
+    <geometry>
+      <mesh filename="file://$(find navexbot_description)/meshes/Wheel_LF_1.stl" scale="0.001 0.001 0.001"/>
+    </geometry>
+  </collision>
+</link>
+<link name="Wheel_LB_1">
+  <inertial>
+    <origin xyz="-0.32305733222430744 -0.6888367667394968 -0.5816959511622183" rpy="0 0 0"/>
+    <mass value="0.037002439542276666"/>
+    <inertia ixx="1.5e-05" iyy="2.5e-05" izz="1.5e-05" ixy="-0.0" iyz="0.0" ixz="0.0"/>
+  </inertial>
+  <visual>
+    <origin xyz="-0.603115 -1.461895 -1.179142" rpy="0 0 0"/>
+    <geometry>
+      <mesh filename="file://$(find navexbot_description)/meshes/Wheel_LB_1.stl" scale="0.001 0.001 0.001"/>
+    </geometry>
+    <material name="silver"/>
+  </visual>
+  <collision>
+    <origin xyz="-0.603115 -1.461895 -1.179142" rpy="0 0 0"/>
+    <geometry>
+      <mesh filename="file://$(find navexbot_description)/meshes/Wheel_LB_1.stl" scale="0.001 0.001 0.001"/>
+    </geometry>
+  </collision>
+</link>
+<link name="Wheel_RF_1">
+  <inertial>
+    <origin xyz="-0.323056979218717 -0.7260449432999149 -0.5816957849999069" rpy="0 0 0"/>
+    <mass value="0.03700239760564051"/>
+    <inertia ixx="1.5e-05" iyy="2.5e-05" izz="1.5e-05" ixy="0.0" iyz="0.0" ixz="0.0"/>
+  </inertial>
+  <visual>
+    <origin xyz="-0.685046 -1.368789 -1.179142" rpy="0 0 0"/>
+    <geometry>
+      <mesh filename="file://$(find navexbot_description)/meshes/Wheel_RF_1.stl" scale="0.001 0.001 0.001"/>
+    </geometry>
+    <material name="silver"/>
+  </visual>
+  <collision>
+    <origin xyz="-0.685046 -1.368789 -1.179142" rpy="0 0 0"/>
+    <geometry>
+      <mesh filename="file://$(find navexbot_description)/meshes/Wheel_RF_1.stl" scale="0.001 0.001 0.001"/>
+    </geometry>
+  </collision>
+</link>
+<link name="Wheel_RB_1">
+  <inertial>
+    <origin xyz="-0.3230573508026159 -0.7260450190347004 -0.5816959431583748" rpy="0 0 0"/>
+    <mass value="0.0370023992249136"/>
+    <inertia ixx="1.5e-05" iyy="2.5e-05" izz="1.5e-05" ixy="0.0" iyz="0.0" ixz="0.0"/>
+  </inertial>
+  <visual>
+    <origin xyz="-0.603115 -1.368789 -1.179142" rpy="0 0 0"/>
+    <geometry>
+      <mesh filename="file://$(find navexbot_description)/meshes/Wheel_RB_1.stl" scale="0.001 0.001 0.001"/>
+    </geometry>
+    <material name="silver"/>
+  </visual>
+  <collision>
+    <origin xyz="-0.603115 -1.368789 -1.179142" rpy="0 0 0"/>
+    <geometry>
+      <mesh filename="file://$(find navexbot_description)/meshes/Wheel_RB_1.stl" scale="0.001 0.001 0.001"/>
     </geometry>
   </collision>
@@ -146,10 +106,10 @@
 <link name="Line_Tracking_Module_1">
   <inertial>
-    <origin xyz="0.5540313035972204 -0.42631351135466095 -0.5444658120038782" rpy="0 0 0"/>
-    <mass value="0.011999979009967758"/>
+    <origin xyz="-0.3104484455904361 -0.7272508096903704 -0.5856112406290825" rpy="0 0 0"/>
+    <mass value="0.011999979009967751"/>
     <inertia ixx="2e-06" iyy="1e-06" izz="3e-06" ixy="-0.0" iyz="0.0" ixz="0.0"/>
   </inertial>
   <visual>
-    <origin xyz="0.460696 -0.427264 -0.542551" rpy="0 0 0"/>
+    <origin xyz="-0.726234 -1.435644 -1.163392" rpy="0 0 0"/>
     <geometry>
       <mesh filename="file://$(find navexbot_description)/meshes/Line_Tracking_Module_1.stl" scale="0.001 0.001 0.001"/>
@@ -158,5 +118,5 @@
   </visual>
   <collision>
-    <origin xyz="0.460696 -0.427264 -0.542551" rpy="0 0 0"/>
+    <origin xyz="-0.726234 -1.435644 -1.163392" rpy="0 0 0"/>
     <geometry>
       <mesh filename="file://$(find navexbot_description)/meshes/Line_Tracking_Module_1.stl" scale="0.001 0.001 0.001"/>
@@ -164,218 +124,258 @@
   </collision>
 </link>
-<link name="Arduino_Mega_v1_1">
-  <inertial>
-    <origin xyz="-0.024846623231800355 0.029164935620271216 0.0028012635578156322" rpy="0 0 0"/>
-    <mass value="0.03699959187591492"/>
-    <inertia ixx="4.2e-05" iyy="1e-05" izz="5.1e-05" ixy="-1e-06" iyz="1e-06" ixz="0.0"/>
-  </inertial>
-  <visual>
-    <origin xyz="-0.021607 0.036831 -0.048908" rpy="0 0 0"/>
-    <geometry>
-      <mesh filename="file://$(find navexbot_description)/meshes/Arduino_Mega_v1_1.stl" scale="0.001 0.001 0.001"/>
-    </geometry>
-    <material name="silver"/>
-  </visual>
-  <collision>
-    <origin xyz="-0.021607 0.036831 -0.048908" rpy="0 0 0"/>
-    <geometry>
-      <mesh filename="file://$(find navexbot_description)/meshes/Arduino_Mega_v1_1.stl" scale="0.001 0.001 0.001"/>
-    </geometry>
-  </collision>
-</link>
-<link name="Expansion_Board_1">
-  <inertial>
-    <origin xyz="-0.08726576052727084 0.08646332521308203 -0.0034230357875419254" rpy="0 0 0"/>
-    <mass value="0.01901859698907641"/>
-    <inertia ixx="6e-06" iyy="5e-06" izz="1e-05" ixy="0.0" iyz="0.0" ixz="-0.0"/>
-  </inertial>
-  <visual>
-    <origin xyz="-0.083115 0.078424 -0.065747" rpy="0 0 0"/>
-    <geometry>
-      <mesh filename="file://$(find navexbot_description)/meshes/Expansion_Board_1.stl" scale="0.001 0.001 0.001"/>
-    </geometry>
-    <material name="silver"/>
-  </visual>
-  <collision>
-    <origin xyz="-0.083115 0.078424 -0.065747" rpy="0 0 0"/>
-    <geometry>
-      <mesh filename="file://$(find navexbot_description)/meshes/Expansion_Board_1.stl" scale="0.001 0.001 0.001"/>
-    </geometry>
-  </collision>
-</link>
-<link name="wheel_1_1">
-  <inertial>
-    <origin xyz="0.4327751903063669 -0.4281664221543372 -0.5405508438975558" rpy="0 0 0"/>
-    <mass value="0.037002404972170014"/>
-    <inertia ixx="1.5e-05" iyy="2.5e-05" izz="1.5e-05" ixy="-0.0" iyz="-0.0" ixz="0.0"/>
-  </inertial>
-  <visual>
-    <origin xyz="0.393843 -0.36047 -0.558301" rpy="0 0 0"/>
-    <geometry>
-      <mesh filename="file://$(find navexbot_description)/meshes/wheel_1_1.stl" scale="0.001 0.001 0.001"/>
-    </geometry>
-    <material name="silver"/>
-  </visual>
-  <collision>
-    <origin xyz="0.393843 -0.36047 -0.558301" rpy="0 0 0"/>
-    <geometry>
-      <mesh filename="file://$(find navexbot_description)/meshes/wheel_1_1.stl" scale="0.001 0.001 0.001"/>
-    </geometry>
-  </collision>
-</link>
-<link name="wheel_4_1">
-  <inertial>
-    <origin xyz="0.5258811943895968 -0.2918523043337162 -0.5405508379440966" rpy="0 0 0"/>
-    <mass value="0.03700242493307289"/>
-    <inertia ixx="1.5e-05" iyy="2.5e-05" izz="1.5e-05" ixy="0.0" iyz="-0.0" ixz="0.0"/>
-  </inertial>
-  <visual>
-    <origin xyz="0.486949 -0.36047 -0.558301" rpy="0 0 0"/>
-    <geometry>
-      <mesh filename="file://$(find navexbot_description)/meshes/wheel_4_1.stl" scale="0.001 0.001 0.001"/>
-    </geometry>
-    <material name="silver"/>
-  </visual>
-  <collision>
-    <origin xyz="0.486949 -0.36047 -0.558301" rpy="0 0 0"/>
-    <geometry>
-      <mesh filename="file://$(find navexbot_description)/meshes/wheel_4_1.stl" scale="0.001 0.001 0.001"/>
-    </geometry>
-  </collision>
-</link>
-<link name="wheel_3_1">
-  <inertial>
-    <origin xyz="0.44394981714587184 -0.2099212285643192 -0.5405509961025838" rpy="0 0 0"/>
-    <mass value="0.03700242493307289"/>
-    <inertia ixx="1.5e-05" iyy="2.5e-05" izz="1.5e-05" ixy="0.0" iyz="-0.0" ixz="0.0"/>
-  </inertial>
-  <visual>
-    <origin xyz="0.486949 -0.278539 -0.558301" rpy="0 0 0"/>
-    <geometry>
-      <mesh filename="file://$(find navexbot_description)/meshes/wheel_3_1.stl" scale="0.001 0.001 0.001"/>
-    </geometry>
-    <material name="silver"/>
-  </visual>
-  <collision>
-    <origin xyz="0.486949 -0.278539 -0.558301" rpy="0 0 0"/>
-    <geometry>
-      <mesh filename="file://$(find navexbot_description)/meshes/wheel_3_1.stl" scale="0.001 0.001 0.001"/>
-    </geometry>
-  </collision>
-</link>
-<link name="wheel_2_1">
-  <inertial>
-    <origin xyz="0.35084381306264295 -0.34623549792373326 -0.5405510020560437" rpy="0 0 0"/>
-    <mass value="0.037002404972170014"/>
-    <inertia ixx="1.5e-05" iyy="2.5e-05" izz="1.5e-05" ixy="-0.0" iyz="-0.0" ixz="0.0"/>
-  </inertial>
-  <visual>
-    <origin xyz="0.393843 -0.278539 -0.558301" rpy="0 0 0"/>
-    <geometry>
-      <mesh filename="file://$(find navexbot_description)/meshes/wheel_2_1.stl" scale="0.001 0.001 0.001"/>
-    </geometry>
-    <material name="silver"/>
-  </visual>
-  <collision>
-    <origin xyz="0.393843 -0.278539 -0.558301" rpy="0 0 0"/>
-    <geometry>
-      <mesh filename="file://$(find navexbot_description)/meshes/wheel_2_1.stl" scale="0.001 0.001 0.001"/>
-    </geometry>
-  </collision>
-</link>
-<link name="C1M1_appearance_V2_20230926.3d_model_v2_1">
-  <inertial>
-    <origin xyz="8.370960599702465e-05 -9.423957307488382e-05 0.013994531625658668" rpy="0 0 0"/>
+<link name="Lidar_1">
+  <inertial>
+    <origin xyz="8.356952260829553e-05 -9.376054348042562e-05 0.013994586411218868" rpy="0 0 0"/>
     <mass value="0.1179926993495319"/>
     <inertia ixx="5.2e-05" iyy="5.2e-05" izz="7.3e-05" ixy="-0.0" iyz="-0.0" ixz="0.0"/>
   </inertial>
   <visual>
-    <origin xyz="-0.045076 -6.4e-05 -0.156908" rpy="0 0 0"/>
-    <geometry>
-      <mesh filename="file://$(find navexbot_description)/meshes/C1M1_appearance_V2_20230926.3d_model_v2_1.stl" scale="0.001 0.001 0.001"/>
-    </geometry>
-    <material name="silver"/>
-  </visual>
-  <collision>
-    <origin xyz="-0.045076 -6.4e-05 -0.156908" rpy="0 0 0"/>
-    <geometry>
-      <mesh filename="file://$(find navexbot_description)/meshes/C1M1_appearance_V2_20230926.3d_model_v2_1.stl" scale="0.001 0.001 0.001"/>
-    </geometry>
-  </collision>
-</link>
-<joint name="Rigid 1" type="fixed">
-  <origin xyz="0.101915 -0.017411 0.048908" rpy="0 0 0"/>
+    <origin xyz="-0.368133 -0.707504 -0.736604" rpy="0 0 0"/>
+    <geometry>
+      <mesh filename="file://$(find navexbot_description)/meshes/Lidar_1.stl" scale="0.001 0.001 0.001"/>
+    </geometry>
+    <material name="silver"/>
+  </visual>
+  <collision>
+    <origin xyz="-0.368133 -0.707504 -0.736604" rpy="0 0 0"/>
+    <geometry>
+      <mesh filename="file://$(find navexbot_description)/meshes/Lidar_1.stl" scale="0.001 0.001 0.001"/>
+    </geometry>
+  </collision>
+</link>
+<link name="Power_Bank_1">
+  <inertial>
+    <origin xyz="-0.31121848988774364 -0.7074930205641167 -0.5656959324503201" rpy="0 0 0"/>
+    <mass value="0.5000878365425067"/>
+    <inertia ixx="0.000613" iyy="0.000213" izz="0.000743" ixy="0.0" iyz="-0.0" ixz="0.0"/>
+  </inertial>
+  <visual>
+    <origin xyz="-0.591189 -1.414945 -1.2743" rpy="0 0 0"/>
+    <geometry>
+      <mesh filename="file://$(find navexbot_description)/meshes/Power_Bank_1.stl" scale="0.001 0.001 0.001"/>
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
Commit message: feat: update configuration and materials for navexbot

File: navexbot_description/urdf/materials.xacro (robot description, xacro)
@@ -6,4 +6,7 @@
 <material name="black">
   <color rgba="0.000 0.000 0.000 1.000"/>
+</material>
+<material name="light black">
+  <color rgba="0.400 0.400 0.400 1.000"/>
 </material>
 <material name="blue">
@@ -22,3 +25,6 @@
   <color rgba="0.388 0.639 0.380 1.000"/>
 </material>
+  <material name="brown">
+    <color rgba="0.8706 0.8118 0.7647 1.0"/>
+  </material>
 </robot>
